Commit message: debuged track_pnp - code cleaning

File: urdf/hog_ir_marker.urdf.xacro (robot description, xacro)
@@ -7,5 +7,5 @@
       <linkName>irm_link</linkName>
       <kl>0.5</kl>
-      <ka>0.001</ka>
+      <ka>0.003</ka>
       <frameId>irm_link</frameId>
     </plugin>

File: urdf/smocap.urdf.xacro (robot description, xacro)
@@ -5,5 +5,5 @@
   <xacro:property name="camera_x" value="1." />
   <xacro:property name="camera_y" value="1." />
-  <xacro:property name="camera_z" value="1.5" />
+  <xacro:property name="camera_z" value="2.9" />
   <xacro:property name="camera_r" value="0.01" />
   <gazebo>
