Commit message: now supporting several cameras - fixed world_to_cam cam_to_world error

File: urdf/camera.urdf.xacro (robot description, xacro)
@@ -1,5 +1,5 @@
 <?xml version="1.0"?>
 <robot name="smocap_camera" xmlns:xacro="http://www.ros.org/wiki/xacro">
- <xacro:macro name="smocap_camera" params="name _x _y _z _rx _ry _rz">
+ <xacro:macro name="smocap_camera" params="name _x _y _z _rx _ry _rz _k1 _k2 _t1 _t2 _k3">
    <xacro:property name="camera_r" value="0.01" />
    <gazebo>
@@ -86,9 +86,9 @@
         <frameName>camera${name}_link</frameName>
         <hackBaseline>0.07</hackBaseline>
-        <distortionK1>0.0</distortionK1>
-        <distortionK2>0.0</distortionK2>
-        <distortionK3>0.0</distortionK3>
-        <distortionT1>0.0</distortionT1>
-        <distortionT2>0.0</distortionT2>
+        <distortionK1>${_k1}</distortionK1>
+        <distortionK2>${_k2}</distortionK2>
+        <distortionT1>${_t1}</distortionT1>
+        <distortionT2>${_t2}</distortionT2>
+        <distortionK3>${_k3}</distortionK3>
       </plugin>
     </sensor>

Commit message: refactoring for multi marker/ multi camera

File: urdf/camera.urdf.xacro (robot description, xacro)
@@ -1,5 +1,5 @@
 <?xml version="1.0"?>
 <robot name="smocap_camera" xmlns:xacro="http://www.ros.org/wiki/xacro">
- <xacro:macro name="smocap_camera" params="name _x _y _z _rx _ry _rz _k1 _k2 _t1 _t2 _k3">
+ <xacro:macro name="smocap_camera" params="name _x _y _z _rx _ry _rz _k1 _k2 _t1 _t2 _k3 _fps">
    <xacro:property name="camera_r" value="0.01" />
    <gazebo>
@@ -60,7 +60,7 @@
   <gazebo reference="camera${name}_link">
     <sensor type="camera" name="camera">
-      <update_rate>30.0</update_rate>
+      <update_rate>${_fps}</update_rate>
       <camera name="${name}">
-        <horizontal_fov>1.12</horizontal_fov>
+        <horizontal_fov>1.15</horizontal_fov>
         <image>
           <width>1600</width>

File: urdf/hog_ir_marker.urdf.xacro (robot description, xacro)
@@ -1,12 +1,15 @@
 <?xml version="1.0"?>
 <robot name="smocap_marker" xmlns:xacro="http://www.ros.org/wiki/xacro">
+  <xacro:arg name="root_link" default="irm_link"/>
+  <xacro:arg name="mesh" default="ir_marker.dae"/>
   <!-- Marker macros -->
   <xacro:include filename="$(find smocap)/urdf/ir_marker.urdf.xacro" />
+  <xacro:ir_marker root_link="$(arg root_link)" mesh="$(arg mesh)"/>
   <gazebo>
     <plugin name="hand_of_god" filename="libgazebo_ros_hand_of_god.so">
-      <linkName>irm_link</linkName>
+      <linkName>$(arg root_link)</linkName>
       <kl>0.5</kl>
       <ka>0.003</ka>
-      <frameId>irm_link</frameId>
+      <frameId>$(arg root_link)</frameId>
     </plugin>
   </gazebo>
@@ -14,6 +17,6 @@
     <plugin name="ground_truth" filename="libgazebo_ros_p3d.so">
       <frameName>world</frameName>
-      <bodyName>irm_link</bodyName>
-      <topicName>smocap/marker_truth</topicName>
+      <bodyName>$(arg root_link)</bodyName>
+      <topicName>smocap/$(arg root_link)_truth</topicName>
       <updateRate>30.0</updateRate>
     </plugin>

File: urdf/ir_marker.urdf.xacro (robot description, xacro)
@@ -7,21 +7,23 @@
   <!-- Inertia macros -->
   <xacro:include filename="$(find smocap)/urdf/inertias.urdf.xacro" />
-  <link name="irm_link">
-    <visual>
-      <origin xyz="0 0 0" rpy="0 0 0"/>
-      <geometry>
-        <!--<box size="${irm_dx} ${irm_dy} ${irm_dz}"/>-->
-        <mesh filename="package://smocap/meshes/ir_marker.dae"/>
-      </geometry>
-    </visual>
-    <collision>
-      <origin xyz="0 0 0" rpy="0 0 0"/>
-      <geometry>
-        <box size="${irm_dx} ${irm_dy} ${irm_dz}"/>
-      </geometry>
-    </collision>
-    <xacro:inertial_cuboid_with_pose mass="${irm_mass}" x_length="${irm_dx}" y_length="${irm_dy}" z_length="${irm_dz}">
-      <origin xyz="0.00  0.00 0" rpy="0 0 0"/>
-    </xacro:inertial_cuboid_with_pose>
-  </link>
+  <xacro:macro name="ir_marker" params="root_link mesh">
+    <link name="${root_link}">
+      <visual>
+	<origin xyz="0 0 0" rpy="0 0 0"/>
+	<geometry>
+          <!--<box size="${irm_dx} ${irm_dy} ${irm_dz}"/>-->
+          <mesh filename="package://smocap/meshes/${mesh}"/>
+	</geometry>
+      </visual>
+      <collision>
+	<origin xyz="0 0 0" rpy="0 0 0"/>
+	<geometry>
+          <box size="${irm_dx} ${irm_dy} ${irm_dz}"/>
+	</geometry>
+      </collision>
+      <xacro:inertial_cuboid_with_pose mass="${irm_mass}" x_length="${irm_dx}" y_length="${irm_dy}" z_length="${irm_dz}">
+	<origin xyz="0.00  0.00 0" rpy="0 0 0"/>
+      </xacro:inertial_cuboid_with_pose>
+    </link>
+  </xacro:macro>
 </robot>

Commit message: added aruco markers in gazebo simulation

File: urdf/camera.urdf.xacro (robot description, xacro)
@@ -1,10 +1,12 @@
 <?xml version="1.0"?>
 <robot name="smocap_camera" xmlns:xacro="http://www.ros.org/wiki/xacro">
- <xacro:macro name="smocap_camera" params="name _x _y _z _rx _ry _rz _k1 _k2 _t1 _t2 _k3 _fps">
+ <xacro:macro name="smocap_camera" params="_cid _root_link _x _y _z _rx _ry _rz _k1 _k2 _t1 _t2 _k3 _fps _static">
    <xacro:property name="camera_r" value="0.01" />
-   <gazebo>
-     <static>true</static>
-   </gazebo>
-   <link name="camera${name}_link">
+   <xacro:if value="${_static}">
+     <gazebo>
+       <static>true</static>
+     </gazebo>
+   </xacro:if>
+   <link name="camera_${_cid}_link">
     <collision>
       <origin xyz="0 0 0" rpy="0 0 0"/>
@@ -27,5 +29,5 @@
       </inertial>
   </link>
-   <link name="camera${name}_optical_frame">
+   <link name="camera_${_cid}_optical_frame">
     <inertial>
       <mass value="0.01"/>
@@ -48,18 +50,18 @@
     </collision>
   </link>
-  <joint name="camera${name}_joint"  type="fixed">
+  <joint name="camera_${_cid}_joint"  type="fixed">
     <origin xyz="${_x} ${_y} ${_z}" rpy="${_rx} ${_ry} ${_rz}" />
-    <parent link="world"/>
-    <child link="camera${name}_link"/>
+    <parent link="${_root_link}"/>
+    <child link="camera_${_cid}_link"/>
   </joint>
-  <joint name="camera${name}_optical_frame_joint" type="fixed">
+  <joint name="camera_${_cid}_optical_frame_joint" type="fixed">
     <origin rpy="${-PI/2} 0.0 ${-PI/2}" xyz="0.0 0.0 0.0"/>
-    <parent link="camera${name}_link"/>
-    <child link="camera${name}_optical_frame"/>
+    <parent link="camera_${_cid}_link"/>
+    <child link="camera_${_cid}_optical_frame"/>
   </joint>
-  <gazebo reference="camera${name}_link">
+  <gazebo reference="camera_${_cid}_link">
     <sensor type="camera" name="camera">
       <update_rate>${_fps}</update_rate>
-      <camera name="${name}">
+      <camera name="${_cid}">
         <horizontal_fov>1.15</horizontal_fov>
         <image>
@@ -70,5 +72,5 @@
         <clip>
           <near>0.02</near>
-          <far>3</far>
+          <far>15</far>
         </clip>
         <noise>
@@ -81,8 +83,8 @@
         <alwaysOn>true</alwaysOn>
         <updateRate>0.0</updateRate>
-        <cameraName>camera${name}</cameraName>
+        <cameraName>camera_${_cid}</cameraName>
         <imageTopicName>image_raw</imageTopicName>
         <cameraInfoTopicName>camera_info</cameraInfoTopicName>
-        <frameName>camera${name}_link</frameName>
+        <frameName>camera_${_cid}_link</frameName>
         <hackBaseline>0.07</hackBaseline>
         <distortionK1>${_k1}</distortionK1>

File: urdf/chessboard.urdf.xacro (robot description, xacro)
@@ -1,43 +1,66 @@
 <?xml version="1.0"?>
 <robot name="smocap_chessboard" xmlns:xacro="http://www.ros.org/wiki/xacro">
-  <xacro:property name="chsbrd_dx" value="1.0" />
-  <xacro:property name="chsbrd_dy" value="1.0" />
-  <xacro:property name="chsbrd_dz" value="0.01" />
+  <xacro:property name="chsbrd_dx"   value="1.0" />
+  <xacro:property name="chsbrd_dy"   value="1.0" />
+  <xacro:property name="chsbrd_dz"   value="0.01" />
   <xacro:property name="chsbrd_mass" value="0.01" />
-  <!-- Inertia macros -->
+  <xacro:property name="chsbrd_z"    value="${-chsbrd_dz/2.}" />  <!-- place origin on face -->
+  <!-- Include inertia macros -->
   <xacro:include filename="$(find smocap)/urdf/inertias.urdf.xacro" />
-  <link name="chessboard_link">
-    <visual>
-      <origin xyz="0 0 0" rpy="0 0 0"/>
-      <geometry>
-        <!--<box size="${chsbrd_dx} ${chsbrd_dy} ${chsbrd_dz}"/>-->
-        <mesh filename="package://smocap/meshes/chessboard.dae"/>
-      </geometry>
-    </visual>
-    <collision>
-      <origin xyz="0 0 0" rpy="0 0 0"/>
-      <geometry>
-        <box size="${chsbrd_dx} ${chsbrd_dy} ${chsbrd_dz}"/>
-      </geometry>
-    </collision>
-    <xacro:inertial_cuboid_with_pose mass="${chsbrd_mass}" x_length="${chsbrd_dx}" y_length="${chsbrd_dy}" z_length="${chsbrd_dz}">
-      <origin xyz="0.00  0.00 0" rpy="0 0 0"/>
-    </xacro:inertial_cuboid_with_pose>
-  </link>
-  <gazebo>
-    <plugin name="hand_of_god" filename="libgazebo_ros_hand_of_god.so">
-      <linkName>chessboard_link</linkName>
-      <kl>0.5</kl>
-      <ka>0.003</ka>
-      <frameId>chessboard_link</frameId>
-    </plugin>
-  </gazebo>
-  <gazebo>
-    <plugin name="ground_truth" filename="libgazebo_ros_p3d.so">
-      <frameName>world</frameName>
-      <bodyName>chessboard_link</bodyName>
-      <topicName>smocap/chessboard_truth</topicName>
-      <updateRate>30.0</updateRate>
-    </plugin>
-  </gazebo>
+  <xacro:macro name="chessboard" params="root_link texture static">
+    <link name="${root_link}">
+      <visual>
+	<origin xyz="0 0 ${chsbrd_z}" rpy="0 0 0"/>
+	<geometry>
+          <box size="${chsbrd_dx} ${chsbrd_dy} ${chsbrd_dz}"/>
+	</geometry>
+      </visual>
+      <collision>
+	<origin xyz="0 0 ${chsbrd_z}" rpy="0 0 0"/>
+	<geometry>
+          <box size="${chsbrd_dx} ${chsbrd_dy} ${chsbrd_dz}"/>
+	</geometry>
+      </collision>
+      <xacro:inertial_cuboid_with_pose mass="${chsbrd_mass}" x_length="${chsbrd_dx}" y_length="${chsbrd_dy}" z_length="${chsbrd_dz}">
+	<origin xyz="0 0 ${chsbrd_z}" rpy="0 0 0"/>
+      </xacro:inertial_cuboid_with_pose>
+    </link>
+    <xacro:property name="bgdx" value="${chsbrd_dx*1.01}"/>
+    <xacro:property name="bgdy" value="${chsbrd_dy*1.01}"/>
+    <xacro:property name="bgdz" value="${chsbrd_dz*1.00}"/>
+    <xacro:property name="bgz"  value="${chsbrd_z-chsbrd_dz*0.1}" />  <!-- move background 10 percent behind chessboard -->
+    <link name="background_link">
+      <visual>
+	<origin xyz="0 0 ${bgz}" rpy="0 0 0"/>
+	<geometry>
+          <box size="${bgdx} ${bgdy} ${bgdz}"/>
+	</geometry>
+      </visual>
+      <collision>
+	<origin xyz="0 0 ${bgz}" rpy="0 0 0"/>
+	<geometry>
+          <box size="${bgdx} ${bgdy} ${bgdz}"/>
+	</geometry>
+      </collision>
+      <xacro:inertial_cuboid_with_pose mass="${chsbrd_mass}" x_length="${bgdx}" y_length="${bgdy}" z_length="${bgdz}">
+	<origin xyz="0 0 ${bgz}" rpy="0 0 0"/>
+      </xacro:inertial_cuboid_with_pose>
+    </link>
+    <joint name="fixed" type="fixed">
+      <parent link="${root_link}"/>
+      <child link="background_link"/>
+    </joint>
+    <gazebo reference="${root_link}">
+      <!--<material>Gazebo/Orange</material>-->
+      <material>${texture}</material>
+    </gazebo>
+    <gazebo reference="background_link">
+      <material>Gazebo/White</material>
+    </gazebo>
+    <xacro:if value="${static}">
+      <gazebo>
+	<static>true</static>
+      </gazebo>
+    </xacro:if>
+  </xacro:macro>
 </robot>

File: urdf/hog_ir_marker.urdf.xacro (robot description, xacro)
@@ -3,4 +3,5 @@
   <xacro:arg name="root_link" default="irm_link"/>
   <xacro:arg name="mesh" default="ir_marker.dae"/>
+  <xacro:arg name="texture" default="unused"/>
   <!-- Marker macros -->
   <xacro:include filename="$(find smocap)/urdf/ir_marker.urdf.xacro" />
@@ -9,5 +10,5 @@
     <plugin name="hand_of_god" filename="libgazebo_ros_hand_of_god.so">
       <linkName>$(arg root_link)</linkName>
-      <kl>0.5</kl>
+      <kl>0.4</kl>
       <ka>0.003</ka>
       <frameId>$(arg root_link)</frameId>
