Commit message: rework : separated mono and multi marker trackers

File: smocap/urdf/camera.urdf.xacro (robot description, xacro)
@@ -1,5 +1,5 @@
 <?xml version="1.0"?>
 <robot name="smocap_camera" xmlns:xacro="http://www.ros.org/wiki/xacro">
- <xacro:macro name="smocap_camera" params="_cid _root_link _x _y _z _rx _ry _rz _k1 _k2 _t1 _t2 _k3 _fps _static">
+ <xacro:macro name="smocap_camera" params="_cid _root_link _x _y _z _rx _ry _rz _w _h _k1 _k2 _t1 _t2 _k3 _fps _static">
    <xacro:property name="camera_r" value="0.01" />
    <xacro:if value="${_static}">
@@ -61,11 +61,11 @@
   </joint>
   <gazebo reference="camera_${_cid}_link">
-    <sensor type="camera" name="camera">
+    <sensor type="camera" name="camera_${_cid}">
       <update_rate>${_fps}</update_rate>
       <camera name="${_cid}">
         <horizontal_fov>1.15</horizontal_fov>
         <image>
-          <width>1600</width>
-          <height>1200</height>
+          <width>${_w}</width>
+          <height>${_h}</height>
           <format>R8G8B8</format>
         </image>

File: smocap/urdf/hog_camera.urdf.xacro (robot description, xacro)
@@ -10,4 +10,6 @@
   <xacro:arg name="camera_P"  default="0."/>
   <xacro:arg name="camera_Y"  default="0."/>
+  <xacro:arg name="camera_w"  default="640"/>
+  <xacro:arg name="camera_h"  default="480"/>
   <xacro:arg name="camera_root_link"  default="camera_root_link"/>
   <!-- Import camera macros -->
@@ -18,4 +20,5 @@
 		       _x="$(arg camera_x)" _y="$(arg camera_y)" _z="$(arg camera_z)"
 		       _rx="$(arg camera_R)" _ry="$(arg camera_P)" _rz="$(arg camera_Y)"
+		       _w="$(arg camera_w)" _h="$(arg camera_h)"
 		       _k1="0." _k2="0." _k3="0." _t1="0." _t2="0." _fps="30." _static="false"/>
   <gazebo>

Commit message: rework

File: smocap/urdf/camera.urdf.xacro (robot description, xacro)
@@ -27,5 +27,5 @@
       <origin xyz="0 0 0" rpy="0 0 0"/>
       <inertia ixx="1e-6" ixy="0" ixz="0" iyy="1e-6" iyz="0" izz="1e-6" />
-      </inertial>
+    </inertial>
   </link>
    <link name="camera_${_cid}_optical_frame">
@@ -64,5 +64,6 @@
       <update_rate>${_fps}</update_rate>
       <camera name="${_cid}">
-        <horizontal_fov>1.15</horizontal_fov>
+        <!-- <horizontal_fov>1.15</horizontal_fov> -->
+        <horizontal_fov>1.2</horizontal_fov>
         <image>
           <width>${_w}</width>

Commit message: improved multimarker

File: smocap/urdf/camera.urdf.xacro (robot description, xacro)
@@ -1,5 +1,5 @@
 <?xml version="1.0"?>
 <robot name="smocap_camera" xmlns:xacro="http://www.ros.org/wiki/xacro">
- <xacro:macro name="smocap_camera" params="_cid _root_link _x _y _z _rx _ry _rz _w _h _k1 _k2 _t1 _t2 _k3 _fps _static">
+ <xacro:macro name="smocap_camera" params="_cid _root_link _x _y _z _rx _ry _rz _w _h _hfov _k1 _k2 _t1 _t2 _k3 _fps _static">
    <xacro:property name="camera_r" value="0.01" />
    <xacro:if value="${_static}">
@@ -8,19 +8,16 @@
      </gazebo>
    </xacro:if>
+   <!-- camera body -->
    <link name="camera_${_cid}_link">
-    <collision>
-      <origin xyz="0 0 0" rpy="0 0 0"/>
-      <geometry>
-	<box size="${camera_r} ${camera_r} ${camera_r}"/>
-      </geometry>
-    </collision>
     <visual>
       <origin xyz="0 0 0" rpy="0 0 0"/>
-      <geometry>
-	<box size="${camera_r} ${camera_r} ${camera_r}"/>
-      </geometry>
+      <geometry><box size="${camera_r} ${camera_r} ${camera_r}"/></geometry>
       <material name="red"/>
       <cast_shadows>false</cast_shadows>
     </visual>
+    <collision>
+      <origin xyz="0 0 0" rpy="0 0 0"/>
+      <geometry><box size="${camera_r} ${camera_r} ${camera_r}"/></geometry>
+    </collision>
     <inertial>
       <mass value="1e-5" />
@@ -29,12 +26,7 @@
     </inertial>
   </link>
+   <!-- camera optical frame -->
    <link name="camera_${_cid}_optical_frame">
-    <inertial>
-      <mass value="0.01"/>
-      <origin rpy="0 0 0" xyz="0 0 0"/>
-      <inertia ixx="0.001" ixy="0.0" ixz="0.0" iyy="0.001" iyz="0.0" izz="0.001"/>
-    </inertial>
-    <visual>
-      <!-- bogus values for visual aesthetics -->
+     <visual>
       <origin rpy="0 0 ${PI/2}" xyz="0 0 0"/>
       <geometry>
@@ -43,4 +35,9 @@
       <material name="Blue"/>
     </visual>
+    <inertial>
+      <mass value="0.01"/>
+      <origin rpy="0 0 0" xyz="0 0 0"/>
+      <inertia ixx="0.001" ixy="0.0" ixz="0.0" iyy="0.001" iyz="0.0" izz="0.001"/>
+    </inertial>
     <collision>
       <origin rpy="0 0 0" xyz="0 0 0"/>
@@ -49,5 +46,5 @@
       </geometry>
     </collision>
-  </link>
+   </link>
   <joint name="camera_${_cid}_joint"  type="fixed">
     <origin xyz="${_x} ${_y} ${_z}" rpy="${_rx} ${_ry} ${_rz}" />
@@ -65,5 +62,5 @@
       <camera name="${_cid}">
         <!-- <horizontal_fov>1.15</horizontal_fov> -->
-        <horizontal_fov>1.2</horizontal_fov>
+        <horizontal_fov>${_hfov}</horizontal_fov>
         <image>
           <width>${_w}</width>
